File: Sofle_Choc/PCB/SofleKeyboard.sch (KiCad schematic (older format))
At the start: 84 parts, among them J2 4PIN, J3 OLED, P1 i2c_pin, P2 i2c_pin, SW1 SW_PUSH_LED, SW10 SW_PUSH_LED, SW11 SW_PUSH_LED, SW12 SW_PUSH_LED, SW13 SW_PUSH_LED, SW14 SW_PUSH_LED, SW15 SW_PUSH_LED, SW16 SW_PUSH_LED, SW17 SW_PUSH_LED, SW18 SW_PUSH_LED, SW19 SW_PUSH_LED, SW2 SW_PUSH_LED, SW20 SW_PUSH_LED, SW21 SW_PUSH_LED, SW22 SW_PUSH_LED, SW23 SW_PUSH_LED, SW24 SW_PUSH_LED, SW25 Rotary_Encoder_Switch, SW26 SW_PUSH_LED, SW27 SW_PUSH_LED, SW28 SW_PUSH_LED, SW29 SW_PUSH_LED, SW3 SW_PUSH_LED, SW30 SW_PUSH_LED, SW4 SW_PUSH_LED, SW5 SW_PUSH_LED, SW6 SW_PUSH_LED, SW7 SW_PUSH_LED, SW8 SW_PUSH_LED, SW9 SW_PUSH_LED, U1 ProMicro

Commit message: Starting backlight
Parts:
- added D31, D32, D33, D34, D35, D36: D, Diode_SMD:D_SOD-123, symbol Diode:1N4148W
- added SW31, SW32, SW33, SW34, SW35, SW36: SW_PUSH_LED, SofleChoc:Choc_Hotswap_SK6812MiniE, symbol SofleKeyboard:SW_PUSH_LED
- D1: footprint Diode_SMD:crkbd-diode -> Diode_SMD:D_SOD-123
- D10, D11, D12, D13, D14, D15, D16, D17, D18, D19, D2, D20, D21, D22, D23, D24, D25, D26, D27, D28, D29, D3, D30, D4, D5, D6, D7, D8, D9: footprint Diode_SMD:crkbd-diode -> Diode_SMD:D_SOD-123; symbol SofleKeyboard-rescue:D-Lily58-cache-Lily58_Pro-rescue -> Diode:1N4148W; Sim.Device (none) -> D; Sim.Pins (none) -> 1=K 2=A
Connections:
- net labels added: row5
- wire segments 162 -> 192
- no-connect marks 3 -> 2
Other:
- moved on the sheet: D1, SW10A, SW10B, SW11A, SW11B, SW12A, SW12B, SW13A, SW13B, SW14A, SW14B, SW15A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
