File: Sofle_Choc/PCB/_autosave-SofleKeyboard.kicad_pcb (KiCad board)
At the start: 2 copper layers, 161.9 x 120.9 mm, 91 parts, among them J2 4PIN, J3 OLED, P1 i2c_pin, P2 i2c_pin, SW1 SW_PUSH_LED, SW10 SW_PUSH_LED, SW11 SW_PUSH_LED, SW12 SW_PUSH_LED, SW13 SW_PUSH_LED, SW14 SW_PUSH_LED, SW15 SW_PUSH_LED, SW16 SW_PUSH_LED, SW17 SW_PUSH_LED, SW18 SW_PUSH_LED, SW19 SW_PUSH_LED, SW2 SW_PUSH_LED, SW20 SW_PUSH_LED, SW21 SW_PUSH_LED, SW22 SW_PUSH_LED, SW23 SW_PUSH_LED, SW24 SW_PUSH_LED, SW25 Rotary_Encoder_Switch, SW26 SW_PUSH_LED, SW27 SW_PUSH_LED, SW28 SW_PUSH_LED, SW29 SW_PUSH_LED, SW3 SW_PUSH_LED, SW30 SW_PUSH_LED, SW31 SW_PUSH_LED, SW32 SW_PUSH_LED, SW33 SW_PUSH_LED, SW4 SW_PUSH_LED, SW5 SW_PUSH_LED, SW6 SW_PUSH_LED, SW7 SW_PUSH_LED, SW8 SW_PUSH_LED, SW9 SW_PUSH_LED, U1 ProMicro

Commit message: Starting backlight
Parts:
- removed G***: LOGO, LOGO
- added D34: SK6812MINI, SofleChoc:SK6812MINI_underglow_dev, F.Cu at (117.8, 59.8)
- added D35: SK6812MINI, SofleChoc:SK6812MINI_underglow_dev, F.Cu at (121.5, 78.8)
- added D36: SK6812MINI, SofleChoc:SK6812MINI_underglow_dev, F.Cu at (120.4, 97.8)
- added D37: SK6812MINI, SofleChoc:SK6812MINI_underglow_dev, F.Cu at (56.6, 4.24)
- added D38: SK6812MINI, SofleChoc:SK6812MINI_underglow_dev, F.Cu at (56.6, 8.89)
- added D39: SK6812MINI, SofleChoc:SK6812MINI_underglow_dev, F.Cu at (56.6, 13.5)
- added D40: SK6812MINI, SofleChoc:SK6812MINI_underglow_dev, F.Cu at (56.6, 18.2)
- added D41: SK6812MINI, SofleChoc:SK6812MINI_underglow_dev, F.Cu at (56.6, 22.8)
- added D42: SK6812MINI, SofleChoc:SK6812MINI_underglow_dev, F.Cu at (167.6, 141.2)
- added D43: SK6812MINI, SofleChoc:SK6812MINI_underglow_dev, F.Cu at (186.0, 146.3)
- added D44: SK6812MINI, SofleChoc:SK6812MINI_underglow_dev, F.Cu at (64.3, 4.24)
- added D46: SK6812MINI, SofleChoc:SK6812MINI_underglow_dev, F.Cu at (64.3, 8.89)
- added D47: SK6812MINI, SofleChoc:SK6812MINI_underglow_dev, F.Cu at (64.3, 13.5)
- added D48: SK6812MINI, SofleChoc:SK6812MINI_underglow_dev, F.Cu at (64.3, 18.2)
- added D49: SK6812MINI, SofleChoc:SK6812MINI_underglow_dev, F.Cu at (64.3, 22.8)
- added D50: SK6812MINI, SofleChoc:SK6812MINI_underglow_dev, F.Cu at (207.7, 23.4)
- added D51: SK6812MINI, SofleChoc:SK6812MINI_underglow_dev, F.Cu at (190.4, 28.1)
- added D52: SK6812MINI, SofleChoc:SK6812MINI_underglow_dev, F.Cu at (72.1, 4.24)
- added D53: SK6812MINI, SofleChoc:SK6812MINI_underglow_dev, F.Cu at (72.1, 8.89)
- added D54: SK6812MINI, SofleChoc:SK6812MINI_underglow_dev, F.Cu at (72.1, 13.5)
Connections:
- SW1 pad 2: Net-(SW1B-DOUT) -> Net-(D34-DIN)
- SW12 pad 2: Net-(SW12B-DOUT) -> Net-(D49-DIN)
- SW12 pad 4: Net-(SW12B-DIN) -> Net-(D48-DOUT)
- SW13 pad 2: Net-(SW13B-DOUT) -> Net-(D36-DIN)
- SW13 pad 4: Net-(SW13B-DIN) -> Net-(D35-DOUT)
- SW18 pad 2: Net-(SW12B-DIN) -> Net-(D48-DIN)
- SW18 pad 4: Net-(SW18B-DIN) -> Net-(D47-DOUT)
- SW19 pad 2: Net-(SW19B-DOUT) -> Net-(D37-DIN)
- SW19 pad 4: Net-(SW13B-DOUT) -> Net-(D36-DOUT)
- SW2 pad 2: Net-(SW2B-DOUT) -> Net-(D54-DIN)
- SW20 pad 4: Net-(SW20B-DIN) -> VCC
- SW22 pad 4: Net-(SW22B-DIN) -> Net-(D43-DOUT)
- SW24 pad 2: Net-(SW18B-DIN) -> Net-(D47-DIN)
- SW24 pad 4: Net-(SW24B-DIN) -> Net-(D46-DOUT)
- SW26 pad 2: Net-(SW20B-DIN) -> Net-(D41-DIN)
- SW26 pad 4: Net-(SW26B-DIN) -> Net-(D40-DOUT)
- SW27 pad 2: Net-(SW27B-DOUT) -> Net-(D42-DIN)
- SW28 pad 2: Net-(SW22B-DIN) -> Net-(D43-DIN)
- SW28 pad 4: Net-(SW27B-DOUT) -> Net-(D42-DOUT)
- SW29 pad 2: Net-(SW29B-DOUT) -> Net-(D44-DIN)
- SW3 pad 4: Net-(SW2B-DOUT) -> Net-(D53-DOUT)
- SW30 pad 2: Net-(SW24B-DIN) -> Net-(D46-DIN)
- SW30 pad 4: Net-(SW29B-DOUT) -> Net-(D44-DOUT)
- SW31 pad 2: Net-(SW31B-DOUT) -> Net-(D38-DIN)
- SW31 pad 4: Net-(SW19B-DOUT) -> Net-(D37-DOUT)
- SW32 pad 2: Net-(SW32B-DOUT) -> Net-(D39-DIN)
- SW32 pad 4: Net-(SW31B-DOUT) -> Net-(D38-DOUT)
- SW33 pad 2: Net-(SW26B-DIN) -> Net-(D40-DIN)
- SW33 pad 4: Net-(SW32B-DOUT) -> Net-(D39-DOUT)
- SW4 pad 2: Net-(SW4B-DOUT) -> Net-(D52-DIN)
- SW5 pad 4: Net-(SW4B-DOUT) -> Net-(D51-DOUT)
- SW6 pad 2: unconnected-(SW6B-DOUT-Pad2) -> Net-(D50-DIN)
- SW6 pad 4: Net-(SW12B-DOUT) -> Net-(D49-DOUT)
- SW7 pad 2: Net-(SW13B-DIN) -> Net-(D35-DIN)
- SW7 pad 4: Net-(SW1B-DOUT) -> Net-(D34-DOUT)
Routing:
- net (no net): track 0.00 -> 729.2 mm, vias 0 -> 32
- net Net-(SW19B-DOUT): track 78.7 -> 0.00 mm, vias 4 -> 0
- net Net-(SW4B-DOUT): track 56.6 -> 0.00 mm, vias 2 -> 0
- net Net-(SW29B-DOUT): track 53.5 -> 0.00 mm, vias 2 -> 0
- net Net-(SW26B-DIN): track 52.5 -> 0.00 mm, vias 2 -> 0
- net Net-(SW27B-DOUT): track 51.7 -> 0.00 mm, vias 2 -> 0
- net Net-(SW32B-DOUT): track 50.5 -> 0.00 mm, vias 2 -> 0
- net Net-(SW2B-DOUT): track 49.3 -> 0.00 mm, vias 2 -> 0
- net Net-(SW31B-DOUT): track 44.1 -> 0.00 mm, vias 2 -> 0
- net VCC: track 975.0 -> 1014.2 mm, vias 40 -> 42
- net Net-(SW12B-DIN): track 38.9 -> 0.00 mm, vias 2 -> 0
- net Net-(SW12B-DOUT): track 38.1 -> 0.00 mm, vias 2 -> 0
- net Net-(SW18B-DIN): track 38.1 -> 0.00 mm, vias 2 -> 0
- net Net-(SW24B-DIN): track 37.7 -> 0.00 mm, vias 2 -> 0
- net Net-(SW22B-DIN): track 37.7 -> 0.00 mm, vias 2 -> 0
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